File: Final_project/Final_project.kicad_sch (KiCad schematic)
At the start: 34 parts, among them J1 USB4105-GF-A, J2 Conn_01x04, J3 DEBUG, J4 LEFT, J5 RIGHT, U1 RP2040, U2 MCP1702T-3302E_CB, U3 W25Q128JV, Y1 12MHz

Commit message: Layout continued, delete header
Parts:
- removed J3: DEBUG, Connector_PinSocket_2.54mm:PinSocket_1x03_P2.54mm_Vertical, symbol Connector_Generic:Conn_01x03
Other:
- note added: "Remove these and add some test points instead? Communication lines and power 3V3, 5V, GND, SCL, SDA, GPIO0, GPIO10-15"
Changed lines of the file:
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@@
-    (stroke (width 0) (type default) (color 0 0 0 0))
-  )
-  (wire (pts (xy 195.58 130.81) (xy 199.39 130.81))
     (stroke (width 0) (type default) (color 0 0 0 0))
   )
@@
   )
   (wire (pts (xy 85.09 189.23) (xy 85.09 190.5))
-    (stroke (width 0) (type default) (color 0 0 0 0))
-  )
-  (wire (pts (xy 195.58 125.73) (xy 199.39 125.73))
     (stroke (width 0) (type default) (color 0 0 0 0))
   )
@@
     (effects (font (size 1.27 1.27) (thickness 0.254) bold) (justify left bottom))
   )
+  (text "Remove these and add some test points instead?\nCommunication lines and power\n3V3, 5V, GND, SCL, SDA, GPIO0, GPIO10-15"
+    (at 166.37 119.38 0)
+    (effects (font (size 1.27 1.27)) (justify left bottom))
+  )
   (text "RP2040 Datasheet\n\n10 SPI1 SCK\n11 SPI1 TX -> MOSI\n12 SPI1 RX -> MISO\n13 SPI1 CSn"
     (at 205.74 66.04 0)
@@
     (effects (font (size 1.27 1.27)) (justify left bottom))
   )
-  (label "SWDIO" (at 195.58 130.81 180)
-    (effects (font (size 1.27 1.27)) (justify right bottom))
-  )
   (label "GPIO0" (at 147.32 41.91 0)
     (effects (font (size 1.27 1.27)) (justify left bottom))
@@
   )
   (label "GPIO23" (at 256.54 116.84 180)
-    (effects (font (size 1.27 1.27)) (justify right bottom))
-  )
-  (label "SWCLK" (at 195.58 125.73 180)
     (effects (font (size 1.27 1.27)) (justify right bottom))
   )
@@
     (pin "2")
   )
-  (symbol (lib_id "Connector_Generic:Conn_01x03") (at 204.47 128.27 0) (unit 1)
-    (in_bom yes) (on_board yes) (fields_autoplaced)
-    (property "Reference" "J3" (id 0) (at 207.01 126.9999 0)
-      (effects (font (size 1.27 1.27)) (justify left))
-    )
-    (property "Value" "DEBUG" (id 1) (at 207.01 129.5399 0)
-      (effects (font (size 1.27 1.27)) (justify left))
-    )
-    (property "Footprint" "Connector_PinSocket_2.54mm:PinSocket_1x03_P2.54mm_Vertical" (id 2) (at 204.47 128.27 0)
-      (effects (font (size 1.27 1.27)) hide)
-    )
-    (property "Datasheet" "~" (id 3) (at 204.47 128.27 0)
-      (effects (font (size 1.27 1.27)) hide)
-    )
-    (pin "1")
-    (pin "2")
-    (pin "3")
-  )
   (symbol (lib_id "power:+3V3") (at 260.35 124.46 90) (unit 1)
     (in_bom yes) (on_board yes) (fields_autoplaced)
@@
     )
     (property "Datasheet" "" (id 3) (at 85.09 153.67 0)
-      (effects (font (size 1.27 1.27)) hide)
-    )
-    (pin "1")
-  )
-  (symbol (lib_id "power:GND") (at 199.39 128.27 270) (unit 1)
-    (in_bom yes) (on_board yes) (fields_autoplaced)
-    (property "Reference" "#PWR0140" (id 0) (at 193.04 128.27 0)
-      (effects (font (size 1.27 1.27)) hide)
-    )
-    (property "Value" "GND" (id 1) (at 195.58 128.2699 90)
-      (effects (font (size 1.27 1.27)) (justify right))
-    )
-    (property "Footprint" "" (id 2) (at 199.39 128.27 0)
-      (effects (font (size 1.27 1.27)) hide)
-    )
-    (property "Datasheet" "" (id 3) (at 199.39 128.27 0)
       (effects (font (size 1.27 1.27)) hide)
     )
@@
       (reference "#PWR0139") (unit 1) (value "GND") (footprint "")
     )
-    (path "/6c1acbe0-069a-4f38-8487-f2c87cc7507e"
-      (reference "#PWR0140") (unit 1) (value "GND") (footprint "")
-    )
     (path "/f6ebf197-355f-4dab-95cc-2cf7a3404249"
       (reference "#PWR0141") (unit 1) (value "GND") (footprint "")
@@
       (reference "J2") (unit 1) (value "Conn_01x04") (footprint "Connector_PinSocket_2.54mm:PinSocket_1x04_P2.54mm_Horizontal")
     )
-    (path "/5fec1192-656f-447e-906e-6fd0f9640d8c"
-      (reference "J3") (unit 1) (value "DEBUG") (footprint "Connector_PinSocket_2.54mm:PinSocket_1x03_P2.54mm_Vertical")
-    )
     (path "/12aa0857-e5d3-4544-bacf-920ce20de984"

Commit message: almost finished layout
Parts:
- added J3: DEBUG, Connector_PinSocket_2.54mm:PinSocket_1x03_P2.54mm_Vertical, symbol Connector_Generic:Conn_01x03
Connections:
- net GND: now also J3.2 (Pin_2)
- net SWCLK: now also J3.1 (Pin_1)
- net SWDIO: now also J3.3 (Pin_3)
Other:
- note removed: "Remove these and add some test points instead? Communication lines and power 3V3, 5V, GND, SCL, SDA, GPIO0, GPIO10-15"
Changed lines of the file:
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@@
+    (stroke (width 0) (type default) (color 0 0 0 0))
+  )
+  (wire (pts (xy 195.58 130.81) (xy 199.39 130.81))
     (stroke (width 0) (type default) (color 0 0 0 0))
   )
@@
   )
   (wire (pts (xy 85.09 189.23) (xy 85.09 190.5))
+    (stroke (width 0) (type default) (color 0 0 0 0))
+  )
+  (wire (pts (xy 195.58 125.73) (xy 199.39 125.73))
     (stroke (width 0) (type default) (color 0 0 0 0))
   )
@@
     (effects (font (size 1.27 1.27) (thickness 0.254) bold) (justify left bottom))
   )
-  (text "Remove these and add some test points instead?\nCommunication lines and power\n3V3, 5V, GND, SCL, SDA, GPIO0, GPIO10-15"
-    (at 166.37 119.38 0)
-    (effects (font (size 1.27 1.27)) (justify left bottom))
-  )
   (text "RP2040 Datasheet\n\n10 SPI1 SCK\n11 SPI1 TX -> MOSI\n12 SPI1 RX -> MISO\n13 SPI1 CSn"
     (at 205.74 66.04 0)
@@
     (effects (font (size 1.27 1.27)) (justify left bottom))
   )
+  (label "SWDIO" (at 195.58 130.81 180)
+    (effects (font (size 1.27 1.27)) (justify right bottom))
+  )
   (label "GPIO0" (at 147.32 41.91 0)
     (effects (font (size 1.27 1.27)) (justify left bottom))
@@
   )
   (label "GPIO23" (at 256.54 116.84 180)
+    (effects (font (size 1.27 1.27)) (justify right bottom))
+  )
+  (label "SWCLK" (at 195.58 125.73 180)
     (effects (font (size 1.27 1.27)) (justify right bottom))
   )
@@
     (pin "2")
   )
+  (symbol (lib_id "Connector_Generic:Conn_01x03") (at 204.47 128.27 0) (unit 1)
+    (in_bom yes) (on_board yes) (fields_autoplaced)
+    (property "Reference" "J3" (id 0) (at 207.01 126.9999 0)
+      (effects (font (size 1.27 1.27)) (justify left))
+    )
+    (property "Value" "DEBUG" (id 1) (at 207.01 129.5399 0)
+      (effects (font (size 1.27 1.27)) (justify left))
+    )
+    (property "Footprint" "Connector_PinSocket_2.54mm:PinSocket_1x03_P2.54mm_Vertical" (id 2) (at 204.47 128.27 0)
+      (effects (font (size 1.27 1.27)) hide)
+    )
+    (property "Datasheet" "~" (id 3) (at 204.47 128.27 0)
+      (effects (font (size 1.27 1.27)) hide)
+    )
+    (pin "1")
+    (pin "2")
+    (pin "3")
+  )
   (symbol (lib_id "power:+3V3") (at 260.35 124.46 90) (unit 1)
     (in_bom yes) (on_board yes) (fields_autoplaced)
@@
     )
     (property "Datasheet" "" (id 3) (at 85.09 153.67 0)
+      (effects (font (size 1.27 1.27)) hide)
+    )
+    (pin "1")
+  )
+  (symbol (lib_id "power:GND") (at 199.39 128.27 270) (unit 1)
+    (in_bom yes) (on_board yes) (fields_autoplaced)
+    (property "Reference" "#PWR0140" (id 0) (at 193.04 128.27 0)
+      (effects (font (size 1.27 1.27)) hide)
+    )
+    (property "Value" "GND" (id 1) (at 195.58 128.2699 90)
+      (effects (font (size 1.27 1.27)) (justify right))
+    )
+    (property "Footprint" "" (id 2) (at 199.39 128.27 0)
+      (effects (font (size 1.27 1.27)) hide)
+    )
+    (property "Datasheet" "" (id 3) (at 199.39 128.27 0)
       (effects (font (size 1.27 1.27)) hide)
     )
@@
       (reference "#PWR0135") (unit 1) (value "GND") (footprint "")
     )
-    (path "/5f380518-a4aa-4cf5-aa47-79ba18474bc7/928ffee1-d6ad-4114-a47b-b3c925c00d43"
-      (reference "#PWR0136") (unit 1) (value "+3V3") (footprint "")
+    (path "/5f380518-a4aa-4cf5-aa47-79ba18474bc7/3a66c6ca-a5f7-44fb-974d-4838a0af20bc"
+      (reference "#PWR0136") (unit 1) (value "+3.3V") (footprint "")
     )
     (path "/9044928e-cf49-4703-b68a-b82a255f3d2f/1894dcc4-ad87-47b6-a39a-56335193bb79"
@@
       (reference "#PWR0139") (unit 1) (value "GND") (footprint "")
     )
+    (path "/6c1acbe0-069a-4f38-8487-f2c87cc7507e"
+      (reference "#PWR0140") (unit 1) (value "GND") (footprint "")
+    )
     (path "/f6ebf197-355f-4dab-95cc-2cf7a3404249"
       (reference "#PWR0141") (unit 1) (value "GND") (footprint "")
@@
       (reference "J2") (unit 1) (value "Conn_01x04") (footprint "Connector_PinSocket_2.54mm:PinSocket_1x04_P2.54mm_Horizontal")
     )
+    (path "/5fec1192-656f-447e-906e-6fd0f9640d8c"
+      (reference "J3") (unit 1) (value "DEBUG") (footprint "Connector_PinSocket_2.54mm:PinSocket_1x03_P2.54mm_Vertical")
+    )
     (path "/12aa0857-e5d3-4544-bacf-920ce20de984"

Commit message: finishing up layout, a few steps remained
Connections:
- net GPIO0: no longer J4.1 (Pin_1)
- net GPIO10: no longer J4.14 (Pin_14)
- net GPIO11: no longer J4.15 (Pin_15)
- net GPIO12: no longer J4.16 (Pin_16)
- net GPIO13: no longer J4.17 (Pin_17)
- net GPIO14: no longer J4.19 (Pin_19)
- net GPIO15: no longer J4.20 (Pin_20)
- no-connect marks 3 -> 10
Changed lines of the file:
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@@
   (no_connect (at 45.72 44.45))
   (no_connect (at 196.85 91.44))
+  (no_connect (at 231.14 147.32))
+  (no_connect (at 231.14 162.56))
+  (no_connect (at 231.14 152.4))
+  (no_connect (at 231.14 154.94))
+  (no_connect (at 231.14 114.3))
+  (no_connect (at 231.14 149.86))
+  (no_connect (at 231.14 160.02))
   (polyline (pts (xy 209.55 140.97) (xy 209.55 162.56))
     (stroke (width 0) (type default) (color 0 0 0 0))
@@
     (effects (font (size 1.27 1.27)) (justify left bottom))
   )
-  (label "GPIO15" (at 231.14 162.56 0)
-    (effects (font (size 1.27 1.27)) (justify left bottom))
-  )
   (label "GPIO6" (at 231.14 134.62 0)
     (effects (font (size 1.27 1.27)) (justify left bottom))
@@
     (effects (font (size 1.27 1.27)) (justify left bottom))
   )
-  (label "GPIO14" (at 231.14 160.02 0)
-    (effects (font (size 1.27 1.27)) (justify left bottom))
-  )
   (label "GPIO11" (at 147.32 97.79 0)
     (effects (font (size 1.27 1.27)) (justify left bottom))
@@
     (effects (font (size 1.27 1.27)) (justify left bottom))
   )
-  (label "GPIO11" (at 231.14 149.86 0)
-    (effects (font (size 1.27 1.27)) (justify left bottom))
-  )
   (label "GPIO27" (at 147.32 179.07 0)
     (effects (font (size 1.27 1.27)) (justify left bottom))
@@
     (effects (font (size 1.27 1.27)) (justify right bottom))
   )
-  (label "GPIO13" (at 231.14 154.94 0)
-    (effects (font (size 1.27 1.27)) (justify left bottom))
-  )
   (label "GPIO21" (at 147.32 148.59 0)
     (effects (font (size 1.27 1.27)) (justify left bottom))
@@
     (effects (font (size 1.27 1.27)) (justify right bottom))
   )
-  (label "GPIO10" (at 231.14 147.32 0)
-    (effects (font (size 1.27 1.27)) (justify left bottom))
-  )
   (label "GPIO5" (at 147.32 67.31 0)
     (effects (font (size 1.27 1.27)) (justify left bottom))
@@
     (effects (font (size 1.27 1.27)) (justify left bottom))
   )
-  (label "GPIO12" (at 231.14 152.4 0)
-    (effects (font (size 1.27 1.27)) (justify left bottom))
-  )
   (label "GPIO29" (at 147.32 189.23 0)
     (effects (font (size 1.27 1.27)) (justify left bottom))
@@
     (effects (font (size 1.27 1.27)) (justify right bottom))
   )
-  (label "GPIO0" (at 231.14 114.3 0)
-    (effects (font (size 1.27 1.27)) (justify left bottom))
-  )
   (label "GPIO26" (at 256.54 137.16 180)

Commit message: Add 3d, fixing vias and layout issues
Parts:
- removed J3: DEBUG, Connector_PinSocket_2.54mm:PinSocket_1x03_P2.54mm_Vertical, symbol Connector_Generic:Conn_01x03
- C1, C2, C3: footprint Final_project:CL10B104JB8NNNC -> Capacitor_SMD:C_0603_1608Metric; Digi-Key_Part (none) -> CL10B104JB8NNNC
- C10, C11, C4, C5, C6, C7: footprint Final_project:CL10B104JB8NNNC -> Capacitor_SMD:C_0603_1608Metric
- C12, C13: footprint Final_project:GRM188R61E106KA73D -> Capacitor_SMD:C_0603_1608Metric; Digi-Key_Part (none) -> GRM188R61E106KA73D
- C8: footprint Final_project:CL10B105KA8NNNC -> Capacitor_SMD:C_0603_1608Metric; Digi-Key_Part (none) -> CL10B105KA8NNNC
- C9: footprint Final_project:CL10B105KA8NNNC -> Capacitor_SMD:C_0603_1608Metric
- R1: footprint Final_project:RES_ERJ3EKF5101V -> Resistor_SMD:R_0603_1608Metric
- R2, R4: footprint Final_project:RES_ERJ3EKF5101V -> Resistor_SMD:R_0603_1608Metric; Digi-Key_Part (none) -> ERJ-3EKF5101V
- R3: footprint Final_project:RES_ERJ3EKF5101V -> Resistor_SMD:R_0603_1608Metric; Digi-Key_Part (none) -> ERJ-3EKF5101VERJ-3EKF5101V
- R5: footprint Final_project:RC0603FR-071KL -> Resistor_SMD:R_0603_1608Metric; Part (none) -> RC0603FR-071KL
- R6: footprint Final_project:RC0603FR-071KL -> Resistor_SMD:R_0603_1608Metric
- R7, R8: footprint Final_project:RC0603FR-071KL -> Resistor_SMD:R_0603_1608Metric; Digi-Key_Part (none) -> RC0603FR-071KL
