File: Final_project/Final_project_no_connector.kicad_pcb (KiCad board)
At the start: 2 copper layers, 65.4 x 29 mm, 54 parts, among them J1 USB4105-GF-A, J2 Conn_01x04, U1 RP2040, U2 MCP1702T-3302E_CB, U3 W25Q128JV, U4 ESP32-WROOM-32, U5 LM393D, Y1 12MHz

Commit message: Complete layout for no connectors add silkscreens
Parts:
- added G***: LOGO, Final_project:dust1, B.Cu at (127.1, 66.3)
- added G***: LOGO, Final_project:dust1, B.Cu at (148.3, 65.8)
- added G***: LOGO, Final_project:ghibli, B.Cu at (152.5, 67.1)
- added G***: LOGO, Final_project:dust1, B.Cu at (95.9, 69.4)
- added G***: LOGO, Final_project:ghibli, B.Cu at (101.2, 67.6)
- added G***: LOGO, Final_project:ghibli, B.Cu at (94.8, 78.7)
- added G***: LOGO, Final_project:ghibli, B.Cu at (94.0, 65.7)
- added G***: LOGO, Final_project:dust1, B.Cu at (99.5, 76.3)
- added G***: LOGO, Final_project:ghibli, B.Cu at (116.4, 67.0)
- added G***: LOGO, Final_project:ghibli, B.Cu at (101.7, 71.6)
- added G***: LOGO, Final_project:dust1, B.Cu at (94.6, 83.7)
- added G***: LOGO, Final_project:ghibli, B.Cu at (109.0, 70.2)
- added G***: LOGO, Final_project:ghibli, B.Cu at (150.3, 70.6)
- added G***: LOGO, Final_project:ghibli, B.Cu at (123.8, 69.6)
- added G***: LOGO, Final_project:ghibli, B.Cu at (95.1, 72.9)
